File: Hardware/mvpUI/misc.kicad_sch (KiCad schematic)
At the start: 35 parts, among them SW10 snap_dome, SW11 snap_dome, SW12 snap_dome, SW13 snap_dome, SW14 snap_dome, SW15 snap_dome, SW16 snap_dome, SW17 snap_dome, SW18 snap_dome, SW3 snap_dome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

Commit message: Getting there...
Just need logic and power planes for the most part (and verify everything once more)
Parts:
- SW10, SW11, SW12, SW13, SW14, SW7, SW8: footprint snap dome:snap dome -> snap dome:snap dome_2
- SW15, SW16, SW17, SW18, SW3, SW4, SW5, SW6, SW9: footprint snap dome:snap dome -> snap dome:snap dome_1
Connections:
- net C0 renamed KEYPAD.C0
- net C1 renamed KEYPAD.C1
- net C2 renamed KEYPAD.C2
- net C3 renamed KEYPAD.C3
- net R0 renamed KEYPAD.R0
- net R1 renamed KEYPAD.R1
- net R2 renamed KEYPAD.R2
- net R3 renamed KEYPAD.R3

Commit message: Getting there part ii
Started power planes, most of keyboard wired together
Parts:
- SW9: footprint snap dome:snap dome_1 -> snap dome:snap dome_2
Changed lines of the file:
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@@
       (effects (font (size 1.27 1.27)))
     )
-    (property "Footprint" "snap dome:snap dome_1" (at 71.12 113.03 0)
+    (property "Footprint" "snap dome:snap dome_2" (at 71.12 113.03 0)
       (effects (font (size 1.27 1.27)) hide)
     )

Commit message: T-2 or 3ish
Just keypad, decaps, and a checkover left!
Parts:
- SW10, SW11, SW12, SW13, SW14, SW15, SW16, SW17, SW18, SW3, SW4, SW5, SW6, SW7, SW8, SW9: now left out of the parts list
Changed lines of the file:
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@@
   )
   (symbol (lib_id "snap dome:snap_dome") (at 118.11 71.12 0) (unit 1)
-    (in_bom yes) (on_board yes) (dnp no) (fields_autoplaced)
+    (in_bom no) (on_board yes) (dnp no) (fields_autoplaced)
     (property "Reference" "SW5" (at 118.11 63.5 0)
       (effects (font (size 1.27 1.27)))
@@
   )
   (symbol (lib_id "snap dome:snap_dome") (at 128.27 53.34 0) (unit 1)
-    (in_bom yes) (on_board yes) (dnp no) (fields_autoplaced)
+    (in_bom no) (on_board yes) (dnp no) (fields_autoplaced)
     (property "Reference" "SW18" (at 128.27 45.72 0)
       (effects (font (size 1.27 1.27)))
@@
   )
   (symbol (lib_id "snap dome:snap_dome") (at 93.98 88.9 0) (unit 1)
-    (in_bom yes) (on_board yes) (dnp no) (fields_autoplaced)
+    (in_bom no) (on_board yes) (dnp no) (fields_autoplaced)
     (property "Reference" "SW7" (at 93.98 81.28 0)
       (effects (font (size 1.27 1.27)))
@@
   )
   (symbol (lib_id "snap dome:snap_dome") (at 93.98 107.95 0) (unit 1)
-    (in_bom yes) (on_board yes) (dnp no) (fields_autoplaced)
+    (in_bom no) (on_board yes) (dnp no) (fields_autoplaced)
     (property "Reference" "SW10" (at 93.98 100.33 0)
       (effects (font (size 1.27 1.27)))
@@
   )
   (symbol (lib_id "snap dome:snap_dome") (at 105.41 53.34 0) (unit 1)
-    (in_bom yes) (on_board yes) (dnp no) (fields_autoplaced)
+    (in_bom no) (on_board yes) (dnp no) (fields_autoplaced)
     (property "Reference" "SW17" (at 105.41 45.72 0)
       (effects (font (size 1.27 1.27)))
@@
   )
   (symbol (lib_id "snap dome:snap_dome") (at 71.12 127 0) (unit 1)
-    (in_bom yes) (on_board yes) (dnp no) (fields_autoplaced)
+    (in_bom no) (on_board yes) (dnp no) (fields_autoplaced)
     (property "Reference" "SW12" (at 71.12 119.38 0)
       (effects (font (size 1.27 1.27)))
@@
   )
   (symbol (lib_id "snap dome:snap_dome") (at 62.23 53.34 0) (unit 1)
-    (in_bom yes) (on_board yes) (dnp no) (fields_autoplaced)
+    (in_bom no) (on_board yes) (dnp no) (fields_autoplaced)
     (property "Reference" "SW15" (at 62.23 45.72 0)
       (effects (font (size 1.27 1.27)))
@@
   )
   (symbol (lib_id "snap dome:snap_dome") (at 71.12 88.9 0) (unit 1)
-    (in_bom yes) (on_board yes) (dnp no) (fields_autoplaced)
+    (in_bom no) (on_board yes) (dnp no) (fields_autoplaced)
     (property "Reference" "SW6" (at 71.12 81.28 0)
       (effects (font (size 1.27 1.27)))
@@
   )
   (symbol (lib_id "snap dome:snap_dome") (at 71.12 107.95 0) (unit 1)
-    (in_bom yes) (on_board yes) (dnp no) (fields_autoplaced)
+    (in_bom no) (on_board yes) (dnp no) (fields_autoplaced)
     (property "Reference" "SW9" (at 71.12 100.33 0)
       (effects (font (size 1.27 1.27)))
@@
   )
   (symbol (lib_id "snap dome:snap_dome") (at 93.98 127 0) (unit 1)
-    (in_bom yes) (on_board yes) (dnp no) (fields_autoplaced)
+    (in_bom no) (on_board yes) (dnp no) (fields_autoplaced)
     (property "Reference" "SW13" (at 93.98 119.38 0)
       (effects (font (size 1.27 1.27)))
@@
   )
   (symbol (lib_id "snap dome:snap_dome") (at 118.11 88.9 0) (unit 1)
-    (in_bom yes) (on_board yes) (dnp no) (fields_autoplaced)
+    (in_bom no) (on_board yes) (dnp no) (fields_autoplaced)
     (property "Reference" "SW8" (at 118.11 81.28 0)
       (effects (font (size 1.27 1.27)))
@@
   )
   (symbol (lib_id "snap dome:snap_dome") (at 118.11 107.95 0) (unit 1)
-    (in_bom yes) (on_board yes) (dnp no) (fields_autoplaced)
+    (in_bom no) (on_board yes) (dnp no) (fields_autoplaced)
     (property "Reference" "SW11" (at 118.11 100.33 0)
       (effects (font (size 1.27 1.27)))
@@
   )
   (symbol (lib_id "snap dome:snap_dome") (at 118.11 127 0) (unit 1)
-    (in_bom yes) (on_board yes) (dnp no) (fields_autoplaced)
+    (in_bom no) (on_board yes) (dnp no) (fields_autoplaced)
     (property "Reference" "SW14" (at 118.11 119.38 0)
       (effects (font (size 1.27 1.27)))
@@
   )
   (symbol (lib_id "snap dome:snap_dome") (at 83.82 53.34 0) (unit 1)
-    (in_bom yes) (on_board yes) (dnp no) (fields_autoplaced)
+    (in_bom no) (on_board yes) (dnp no) (fields_autoplaced)
     (property "Reference" "SW16" (at 83.82 45.72 0)
       (effects (font (size 1.27 1.27)))
@@
   )
   (symbol (lib_id "snap dome:snap_dome") (at 93.98 71.12 0) (unit 1)
-    (in_bom yes) (on_board yes) (dnp no) (fields_autoplaced)
+    (in_bom no) (on_board yes) (dnp no) (fields_autoplaced)
     (property "Reference" "SW4" (at 93.98 63.5 0)
       (effects (font (size 1.27 1.27)))
@@
   )
   (symbol (lib_id "snap dome:snap_dome") (at 71.12 71.12 0) (unit 1)
-    (in_bom yes) (on_board yes) (dnp no) (fields_autoplaced)
+    (in_bom no) (on_board yes) (dnp no) (fields_autoplaced)
     (property "Reference" "SW3" (at 71.12 63.5 0)
       (effects (font (size 1.27 1.27)))
