File: Hardware/mvpUI/mcu.kicad_sch (KiCad schematic)
At the start: 31 parts, among them J1 Conn_ARM_SWD_TagConnect_TC203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, SW1 SW_Push, U1 MX25R3235FM2xx0, U8 STM32U585VIT6Q, Y1 16Mhz, Y2 Crystal

Commit message: Getting there...
Just need logic and power planes for the most part (and verify everything once more)
Parts:
- added C1: 10uF, Capacitor_SMD_US_Handsoldering_AKL:C_0603_1608Metric, symbol Device:C
- added C2: 100nF, Capacitor_SMD_US_Handsoldering_AKL:C_0603_1608Metric, symbol Device:C
- added J3: MEM2061-01-188-00-A_REVA, phone:GCT_MEM2061-01-188-00-A_REVA, symbol MEM2061-01-188-00-A_REVA:MEM2061-01-188-00-A_REVA
- C23, C28, Y1: now not fitted; now left out of the parts list
Connections:
- net +3.3V: now also C1.1, C2.1, J3.4 (VDD)
- net GND: now also C1.2, C2.2, J3.10 (CD2), J3.11 (GND), J3.12 (GND__1), J3.6 (VSS), J3.9 (CD1)
- net SD_CLK: now also J3.5 (CLK)
- net SD_CMD: now also J3.3 (CMD)
- net SD_IO0: now also J3.7 (DAT0)
- net SD_IO1: now also J3.8 (DAT1)
- net SD_IO2: now also J3.1 (DAT2)
- net SD_IO3: now also J3.2 (CD/DAT3)
- net SWCLK: now also RN1.2 (R2.1); no longer RN1.1 (R1.1)
- net SWDIO: now also RN1.1 (R1.1); no longer RN1.2 (R2.1)
Other:
- moved on the sheet: J1, RN1

Commit message: Getting there part ii
Started power planes, most of keyboard wired together
Connections:
- net INT: now also U8.96 (PB9); no longer U8.93 (PB7)
- net SDA: now also U8.93 (PB7); no longer U8.89 (PB3)

Commit message: T-2 or 3ish
Just keypad, decaps, and a checkover left!
Connections:
- net B0: now also U8.88 (PD7)
- net B1: now also U8.17 (PC2)
- net BCK: now also U8.7 (PC13)
- net BSP: now also U8.97 (PE0)
- net G0: now also U8.89 (PB3)
- net G1: now also U8.16 (PC1)
- net GCK: now also U8.4 (PE5)
- net GEN: now also U8.2 (PE3)
- net GSP: now also U8.3 (PE4)
- net INTB: now also U8.5 (PE6)
- net R0: now also U8.90 (PB4)
- net R1: now also U8.15 (PC0)
- net VCOM: now also U8.1 (PE2)
Changed lines of the file:
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@@
+    (stroke (width 0) (type default))
+  )
+  (wire (pts (xy 46.99 138.43) (xy 40.64 138.43))
     (stroke (width 0) (type default))
   )
@@
     (stroke (width 0) (type default))
   )
+  (wire (pts (xy 102.87 168.91) (xy 109.22 168.91))
+    (stroke (width 0) (type default))
+  )
   (wire (pts (xy 114.3 64.77) (xy 102.87 64.77))
     (stroke (width 0) (type default))
@@
     (stroke (width 0) (type default))
   )
+  (wire (pts (xy 46.99 87.63) (xy 40.64 87.63))
+    (stroke (width 0) (type default))
+  )
   (bus (pts (xy 149.86 101.6) (xy 149.86 104.14))
     (stroke (width 0) (type default))
@@
     (stroke (width 0) (type default))
   )
+  (wire (pts (xy 102.87 143.51) (xy 109.22 143.51))
+    (stroke (width 0) (type default))
+  )
   (wire (pts (xy 184.15 117.475) (xy 193.675 117.475))
     (stroke (width 0) (type default))
@@
     (stroke (width 0) (type default))
   )
+  (wire (pts (xy 102.87 107.95) (xy 109.22 107.95))
+    (stroke (width 0) (type default))
+  )
   (wire (pts (xy 193.675 127.635) (xy 193.675 132.715))
     (stroke (width 0) (type default))
@@
     (stroke (width 0) (type default))
   )
+  (wire (pts (xy 46.99 92.71) (xy 40.64 92.71))
+    (stroke (width 0) (type default))
+  )
   (wire (pts (xy 111.76 171.45) (xy 102.87 171.45))
     (stroke (width 0) (type default))
@@
     (stroke (width 0) (type default))
   )
+  (wire (pts (xy 46.99 90.17) (xy 40.64 90.17))
+    (stroke (width 0) (type default))
+  )
   (wire (pts (xy 160.02 64.77) (xy 166.37 64.77))
     (stroke (width 0) (type default))
@@
     (stroke (width 0) (type default))
   )
+  (wire (pts (xy 46.99 80.01) (xy 40.64 80.01))
+    (stroke (width 0) (type default))
+  )
   (wire (pts (xy 275.59 58.42) (xy 269.24 58.42))
     (stroke (width 0) (type default))
@@
     (stroke (width 0) (type default))
   )
+  (wire (pts (xy 46.99 85.09) (xy 40.64 85.09))
+    (stroke (width 0) (type default))
+  )
   (wire (pts (xy 114.3 92.71) (xy 102.87 92.71))
     (stroke (width 0) (type default))
@@
     (stroke (width 0) (type default))
   )
+  (wire (pts (xy 102.87 110.49) (xy 109.22 110.49))
+    (stroke (width 0) (type default))
+  )
   (wire (pts (xy 163.195 129.54) (xy 164.465 129.54))
     (stroke (width 0) (type default))
@@
     (stroke (width 0) (type default))
   )
+  (wire (pts (xy 46.99 82.55) (xy 40.64 82.55))
+    (stroke (width 0) (type default))
+  )
   (wire (pts (xy 63.5 12.7) (xy 63.5 0))
     (stroke (width 0) (type default))
@@
     (stroke (width 0) (type default))
   )
+  (wire (pts (xy 102.87 140.97) (xy 109.22 140.97))
+    (stroke (width 0) (type default))
+  )
   (wire (pts (xy 275.59 60.96) (xy 269.24 60.96))
     (stroke (width 0) (type default))
@@
     (stroke (width 0) (type default))
   )
+  (wire (pts (xy 102.87 146.05) (xy 109.22 146.05))
+    (stroke (width 0) (type default))
+  )
   (bus (pts (xy 277.495 143.51) (xy 277.495 146.05))
     (stroke (width 0) (type default))
@@
     (effects (font (size 1.27 1.27)) (justify left bottom))
   )
+  (label "G1" (at 109.22 143.51 180) (fields_autoplaced)
+    (effects (font (size 1.27 1.27)) (justify right bottom))
+  )
   (label "~{CE}" (at 110.49 120.65 180) (fields_autoplaced)
     (effects (font (size 1.27 1.27)) (justify right bottom))
@@
     (effects (font (size 1.27 1.27)) (justify left bottom))
   )
+  (label "B0" (at 40.64 138.43 0) (fields_autoplaced)
+    (effects (font (size 1.27 1.27)) (justify left bottom))
+  )
   (label "KEYPAD.C2" (at 262.255 151.13 0)
     (effects (font (size 1.27 1.27)) (justify left bottom))
@@
     (effects (font (size 1.27 1.27)) (justify right bottom))
   )
+  (label "BCK" (at 109.22 168.91 180) (fields_autoplaced)
+    (effects (font (size 1.27 1.27)) (justify right bottom))
+  )
+  (label "GEN" (at 40.64 85.09 0) (fields_autoplaced)
+    (effects (font (size 1.27 1.27)) (justify left bottom))
+  )
   (label "QSPI_IO3" (at 190.5 40.64 0) (fields_autoplaced)
     (effects (font (size 1.27 1.27)) (justify left bottom))
@@
     (effects (font (size 1.27 1.27)) (justify right bottom))
   )
+  (label "G0" (at 109.22 107.95 180) (fields_autoplaced)
+    (effects (font (size 1.27 1.27)) (justify right bottom))
+  )
   (label "QSPI_CLK" (at 114.3 64.77 180) (fields_autoplaced)
     (effects (font (size 1.27 1.27)) (justify right bottom))
@@
     (effects (font (size 1.27 1.27)) (justify left bottom))
   )
+  (label "BSP" (at 40.64 80.01 0) (fields_autoplaced)
+    (effects (font (size 1.27 1.27)) (justify left bottom))
+  )
+  (label "GSP" (at 40.64 87.63 0) (fields_autoplaced)
+    (effects (font (size 1.27 1.27)) (justify left bottom))
+  )
   (label "SD_CMD" (at 38.1 125.73 0) (fields_autoplaced)
     (effects (font (size 1.27 1.27)) (justify left bottom))
@@
     (effects (font (size 1.27 1.27)) (justify right bottom))
   )
+  (label "VCOM" (at 40.64 82.55 0) (fields_autoplaced)
+    (effects (font (size 1.27 1.27)) (justify left bottom))
+  )
   (label "KEYPAD.C0" (at 262.255 146.05 0)
     (effects (font (size 1.27 1.27)) (justify left bottom))
@@
     (effects (font (size 1.27 1.27)) (justify right bottom))
   )
+  (label "R1" (at 109.22 140.97 180) (fields_autoplaced)
+    (effects (font (size 1.27 1.27)) (justify right bottom))
+  )
   (label "SD_IO0" (at 184.15 112.395 0) (fields_autoplaced)
     (effects (font (size 1.27 1.27)) (justify left bottom))
@@
     (effects (font (size 1.27 1.27)) (justify left bottom))
   )
+  (label "INTB" (at 40.64 92.71 0) (fields_autoplaced)
+    (effects (font (size 1.27 1.27)) (justify left bottom))
+  )
   (label "BCK" (at 269.24 50.8 0) (fields_autoplaced)
     (effects (font (size 1.27 1.27)) (justify left bottom))
@@
     (effects (font (size 1.27 1.27)) (justify left bottom))
   )
+  (label "GCK" (at 40.64 90.17 0) (fields_autoplaced)
+    (effects (font (size 1.27 1.27)) (justify left bottom))
+  )
   (label "~{CE}" (at 160.02 88.9 180) (fields_autoplaced)
     (effects (font (size 1.27 1.27)) (justify right bottom))
@@
     (effects (font (size 1.27 1.27)) (justify left bottom))
   )
+  (label "B1" (at 109.22 146.05 180) (fields_autoplaced)
+    (effects (font (size 1.27 1.27)) (justify right bottom))
+  )
   (label "KEYPAD.R2" (at 262.255 161.29 0)
     (effects (font (size 1.27 1.27)) (justify left bottom))
@@
     (effects (font (size 1.27 1.27)) (justify right bottom))
   )
+  (label "R0" (at 109.22 110.49 180) (fields_autoplaced)
+    (effects (font (size 1.27 1.27)) (justify right bottom))
+  )

Commit message: Ready to Review
Connections:
- net KEYPAD.C0: now also U8.81 (PD0)
- net KEYPAD.C1: now also U8.82 (PD1)
- net KEYPAD.C2: now also U8.23 (PA1)
- net KEYPAD.C3: now also U8.22 (PA0)
- net KEYPAD.R0: now also U8.43 (PE15)
- net KEYPAD.R1: now also U8.52 (PB13)
- net KEYPAD.R2: now also U8.45 (PB11)
- net KEYPAD.R3: now also U8.44 (PB10)
- net MAG1_OUT: now also U8.18 (PC3)
- net SWO: now reaches J1.6 (SWO), RN1.3 (R3.1)
Changed lines of the file:
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@@
+    (stroke (width 0) (type default))
+  )
+  (wire (pts (xy 34.29 115.57) (xy 46.99 115.57))
     (stroke (width 0) (type default))
   )
@@
     (stroke (width 0) (type default))
   )
+  (wire (pts (xy 115.57 125.73) (xy 102.87 125.73))
+    (stroke (width 0) (type default))
+  )
   (wire (pts (xy 274.955 148.59) (xy 262.255 148.59))
     (stroke (width 0) (type default))
@@
     (stroke (width 0) (type default))
   )
+  (wire (pts (xy 34.29 120.65) (xy 46.99 120.65))
+    (stroke (width 0) (type default))
+  )
   (wire (pts (xy 160.02 64.77) (xy 166.37 64.77))
     (stroke (width 0) (type default))
@@
     (stroke (width 0) (type default))
   )
+  (wire (pts (xy 46.99 123.19) (xy 34.29 123.19))
+    (stroke (width 0) (type default))
+  )
   (wire (pts (xy 77.47 45.72) (xy 77.47 49.53))
     (stroke (width 0) (type default))
@@
     (stroke (width 0) (type default))
   )
+  (wire (pts (xy 115.57 57.15) (xy 102.87 57.15))
+    (stroke (width 0) (type default))
+  )
   (wire (pts (xy 48.26 45.72) (xy 48.26 53.34))
     (stroke (width 0) (type default))
@@
     (stroke (width 0) (type default))
   )
+  (wire (pts (xy 115.57 59.69) (xy 102.87 59.69))
+    (stroke (width 0) (type default))
+  )
+  (wire (pts (xy 115.57 130.81) (xy 102.87 130.81))
+    (stroke (width 0) (type default))
+  )
   (wire (pts (xy 102.87 85.09) (xy 111.125 85.09))
     (stroke (width 0) (type default))
@@
     (stroke (width 0) (type default))
   )
+  (wire (pts (xy 115.57 128.27) (xy 102.87 128.27))
+    (stroke (width 0) (type default))
+  )
   (text "SWD" (at 163.195 158.75 0)
     (effects (font (size 1.27 1.27)) (justify left bottom))
@@
     (effects (font (size 1.27 1.27)) (justify left bottom))
   )
+  (label "KEYPAD.C3" (at 115.57 57.15 180) (fields_autoplaced)
+    (effects (font (size 1.27 1.27)) (justify right bottom))
+  )
   (label "KEYPAD.R0" (at 262.255 156.21 0)
     (effects (font (size 1.27 1.27)) (justify left bottom))
@@
     (effects (font (size 1.27 1.27)) (justify left bottom))
   )
+  (label "KEYPAD.C0" (at 34.29 120.65 0) (fields_autoplaced)
+    (effects (font (size 1.27 1.27)) (justify left bottom))
+  )
   (label "QSPI_IO3" (at 190.5 40.64 0) (fields_autoplaced)
     (effects (font (size 1.27 1.27)) (justify left bottom))
@@
     (effects (font (size 1.27 1.27)) (justify left bottom))
   )
+  (label "SWO" (at 158.75 152.4 180) (fields_autoplaced)
+    (effects (font (size 1.27 1.27)) (justify right bottom))
+  )
   (label "KEYPAD.R3" (at 262.255 163.83 0)
     (effects (font (size 1.27 1.27)) (justify left bottom))
@@
     (effects (font (size 1.27 1.27)) (justify right bottom))
   )
+  (label "KEYPAD.C2" (at 115.57 59.69 180) (fields_autoplaced)
+    (effects (font (size 1.27 1.27)) (justify right bottom))
+  )
   (label "LSE_OUT" (at 182.88 54.61 180) (fields_autoplaced)
     (effects (font (size 1.27 1.27)) (justify right bottom))
@@
     (effects (font (size 1.27 1.27)) (justify left bottom))
   )
+  (label "KEYPAD.R2" (at 115.57 128.27 180) (fields_autoplaced)
+    (effects (font (size 1.27 1.27)) (justify right bottom))
+  )
   (label "G1" (at 269.24 71.12 0) (fields_autoplaced)
     (effects (font (size 1.27 1.27)) (justify left bottom))
@@
     (effects (font (size 1.27 1.27)) (justify right bottom))
   )
+  (label "KEYPAD.R1" (at 115.57 130.81 180) (fields_autoplaced)
+    (effects (font (size 1.27 1.27)) (justify right bottom))
+  )
   (label "R1" (at 109.22 140.97 180) (fields_autoplaced)
     (effects (font (size 1.27 1.27)) (justify right bottom))
@@
     (effects (font (size 1.27 1.27)) (justify left bottom))
   )
+  (label "KEYPAD.R3" (at 115.57 125.73 180) (fields_autoplaced)
+    (effects (font (size 1.27 1.27)) (justify right bottom))
+  )
   (label "KEYPAD.C3" (at 262.255 153.67 0)
     (effects (font (size 1.27 1.27)) (justify left bottom))
@@
     (effects (font (size 1.27 1.27)) (justify left bottom))
   )
+  (label "KEYPAD.R0" (at 34.29 115.57 0) (fields_autoplaced)
+    (effects (font (size 1.27 1.27)) (justify left bottom))
+  )
   (label "G0" (at 269.24 68.58 0) (fields_autoplaced)
     (effects (font (size 1.27 1.27)) (justify left bottom))
@@
   (label "SD_IO2" (at 111.76 161.29 180) (fields_autoplaced)
     (effects (font (size 1.27 1.27)) (justify right bottom))
+  )
+  (label "KEYPAD.C1" (at 34.29 123.19 0) (fields_autoplaced)
+    (effects (font (size 1.27 1.27)) (justify left bottom))
   )
   (label "R0" (at 109.22 110.49 180) (fields_autoplaced)
@@
     (effects (font (size 1.27 1.27)) (justify left))
   )
-  (hierarchical_label "MAG1_OUT" (shape input) (at 129.54 121.92 0) (fields_autoplaced)
+  (hierarchical_label "MAG1_OUT" (shape input) (at 102.87 148.59 0) (fields_autoplaced)
     (effects (font (size 1.27 1.27)) (justify left))
   )

Commit message: Production!
Forgot to commit the final, lets hope this works. Also start on software using Slint. Prototype in Plasticity on a free trial to test.
Parts:
- C10, C12, C2, C27, C6, C8, C9: value 100nF -> 0.1uF
- C34: value 100nF X7R -> 0.1uF X7R
Connections:
- no-connect marks 0 -> 29
Changed lines of the file:
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@@
   (junction (at 149.86 31.75) (diameter 0) (color 0 0 0 0)
   )
+  (no_connect (at 46.99 97.79))
+  (no_connect (at 46.99 105.41))
+  (no_connect (at 46.99 113.03))
+  (no_connect (at 46.99 140.97))
+  (no_connect (at 46.99 102.87))
+  (no_connect (at 46.99 146.05))
+  (no_connect (at 102.87 105.41))
+  (no_connect (at 46.99 148.59))
+  (no_connect (at 46.99 107.95))
+  (no_connect (at 46.99 74.93))
+  (no_connect (at 102.87 77.47))
+  (no_connect (at 46.99 128.27))
+  (no_connect (at 102.87 82.55))
+  (no_connect (at 46.99 130.81))
+  (no_connect (at 46.99 156.21))
+  (no_connect (at 46.99 158.75))
+  (no_connect (at 46.99 143.51))
+  (no_connect (at 46.99 153.67))
+  (no_connect (at 102.87 153.67))
+  (no_connect (at 102.87 151.13))
+  (no_connect (at 46.99 133.35))
+  (no_connect (at 102.87 80.01))
+  (no_connect (at 46.99 135.89))
+  (no_connect (at 46.99 110.49))
+  (no_connect (at 46.99 151.13))
+  (no_connect (at 102.87 67.31))
+  (no_connect (at 46.99 100.33))
+  (no_connect (at 46.99 95.25))
+  (no_connect (at 102.87 69.85))
   (bus_entry (at 149.86 101.6) (size 2.54 2.54)
     (stroke (width 0) (type default))
@@
       (effects (font (size 1.27 1.27)) (justify left))
     )
-    (property "Value" "100nF" (at 60.96 -17.78 0)
+    (property "Value" "0.1uF" (at 60.96 -17.78 0)
       (effects (font (size 1.27 1.27)) (justify left))
     )
@@
       (effects (font (size 1.27 1.27)) (justify left))
     )
-    (property "Value" "100nF" (at 60.96 22.86 0)
+    (property "Value" "0.1uF" (at 60.96 22.86 0)
       (effects (font (size 1.27 1.27)) (justify left))
     )
@@
       (effects (font (size 1.27 1.27)) (justify left))
     )
-    (property "Value" "100nF" (at 60.96 -3.81 0)
+    (property "Value" "0.1uF" (at 60.96 -3.81 0)
       (effects (font (size 1.27 1.27)) (justify left))
     )
@@
       (effects (font (size 1.27 1.27)) (justify left))
     )
-    (property "Value" "100nF" (at 60.96 -30.48 0)
+    (property "Value" "0.1uF" (at 60.96 -30.48 0)
       (effects (font (size 1.27 1.27)) (justify left))
     )
@@
       (effects (font (size 1.27 1.27)))
     )
-    (property "Value" "100nF X7R" (at 227.33 43.18 90)
+    (property "Value" "0.1uF X7R" (at 227.33 43.18 90)
       (effects (font (size 1.27 1.27)))
     )
@@
       (effects (font (size 1.27 1.27)) (justify left))
     )
-    (property "Value" "100nF" (at 104.14 22.86 0)
+    (property "Value" "0.1uF" (at 104.14 22.86 0)
       (effects (font (size 1.27 1.27)) (justify left))
     )
@@
       (effects (font (size 1.27 1.27)) (justify left))
     )
-    (property "Value" "100nF" (at 87.63 22.86 0)
+    (property "Value" "0.1uF" (at 87.63 22.86 0)
       (effects (font (size 1.27 1.27)) (justify left))
     )
@@
       (effects (font (size 1.27 1.27)) (justify left))
     )
-    (property "Value" "100nF" (at 119.38 41.91 0)
+    (property "Value" "0.1uF" (at 119.38 41.91 0)
       (effects (font (size 1.27 1.27)) (justify left))
     )
@@
       (effects (font (size 1.27 1.27)) (justify left))
     )
-    (property "Value" "100nF" (at 208.28 97.7899 0)
+    (property "Value" "0.1uF" (at 208.28 97.7899 0)
       (effects (font (size 1.27 1.27)) (justify left))
     )
@@
       (effects (font (size 1.27 1.27)) (justify left))
     )
-    (property "Value" "100nF" (at 60.96 8.89 0)
-      (effects (font (size 1.27 1.27)) (justify left))
-    )
+    (property "Value" "0.1uF" (at 60.96 8.89 0)
+      (effects (font (size 1.27 1.27)) (justify left))
+    )
