File: Hardware/mvpUI/mvpUI.kicad_pcb (KiCad board)
At the start: 4 copper layers, 44 x 108.8 mm, 105 parts, among them IC1 XC9265B331MR-G, J1 Conn_ARM_SWD_TagConnect_TC203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, J2 54-00305, J3 MEM2061-01-188-00-A_REVA, J4 503566-2102, SW1 SW_Push, SW10 snap_dome, SW11 snap_dome, SW12 snap_dome, SW13 snap_dome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

Commit message: Getting there...
Just need logic and power planes for the most part (and verify everything once more)
Parts:
- removed C23, C28: 6.8pF, Capacitor_SMD_US_Handsoldering_AKL:C_0603_1608Metric
- removed Y1: 16Mhz, Crystal_Handsoldering_AKL:Crystal_SMD_3225-4Pin_3.2x2.5mm_BigPads
- added R2: 10k, Resistor_SMD_AKL:R_0603_1608Metric_Pad1.05x0.95mm_HandSolder, F.Cu at (1.71, 0.76)
- C3, C4, C47: moved to B.Cu
- SW10, SW11, SW12, SW13, SW14, SW7, SW8: footprint snap dome:snap dome -> snap dome:snap dome_2
- SW15, SW16, SW17, SW18, SW3, SW4, SW5, SW6, SW9: footprint snap dome:snap dome -> snap dome:snap dome_1
- moved C35 111.2 mm to (104.5, 69.4), turned to 180 degrees
- moved C3 103.3 mm to (112.2, 65.5), turned to 90 degrees
- moved C4 103.0 mm to (112.2, 69.5), turned to -90 degrees
- moved C17 92.3 mm to (124.8, 66.4)
- moved C18 92.3 mm to (124.8, 69.1)
- moved C21 92.3 mm to (129.2, 61.0)
- moved C16 72.1 mm to (109.5, 120.9)
- moved C19 67.5 mm to (107.8, 110.9), turned to 180 degrees
- moved C55 22.2 mm to (90.6, 133.3), turned to -90 degrees
- moved C54 22.0 mm to (88.9, 134.5), turned to -90 degrees
- moved Y2 5.22 mm to (85.5, 108.7), turned to 45 degrees
- moved C30 2.90 mm to (82.6, 107.5), turned to 135 degrees
- moved SW13 2.81 mm to (98.6, 134.3), turned to 170 degrees
- moved RN2 2.55 mm to (83.7, 139.7)
- moved SW12 2.18 mm to (112.0, 133.9), turned to 0 degrees
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Connections:
- net /Misc/C0 renamed /MCU/KEYPAD.C0
- net /Misc/C1 renamed /MCU/KEYPAD.C1
- net /Misc/C2 renamed /MCU/KEYPAD.C2
- net /Misc/C3 renamed /MCU/KEYPAD.C3
- net /Misc/R0 renamed /MCU/KEYPAD.R0
- net /Misc/R1 renamed /MCU/KEYPAD.R1
- net /Misc/R2 renamed /MCU/KEYPAD.R2
- net /Misc/R3 renamed /MCU/KEYPAD.R3
- C39 pad 1: /MCU/VBUS -> /Connectors/VBUS
- C44 pad 1: /Power/V+ -> /Connectors/V+
- J3 pad 1: /Connectors/SDIO.SD_IO2 -> /MCU/SD_IO2
- J3 pad 2: /Connectors/SDIO.SD_IO3 -> /MCU/SD_IO3
- J3 pad 3: /Connectors/SD_CMD -> /MCU/SD_CMD
- J3 pad 5: /Connectors/SD_CLK -> /MCU/SD_CLK
- J3 pad 7: /Connectors/SDIO.SD_IO0 -> /MCU/SD_IO0
- J3 pad 8: /Connectors/SDIO.SD_IO1 -> /MCU/SD_IO1
- R4 pad 2: /Power/TEMP -> /Connectors/TEMP
- R5 pad 2: /Power/TEMP -> /Connectors/TEMP
- RN1 pad 1: /Power/SCL -> /MCU/SCL
- RN1 pad 2: /Power/SDA -> /MCU/SDA
- RN1 pad 3: /Power/INT -> /MCU/INT
- RN1 pad 4: Net-(RN1-R4.1) -> unconnected-(RN1-R4.1-Pad4)
- RN2 pad 1: /MCU/SWCLK -> /MCU/SWDIO
- RN2 pad 2: /MCU/SWDIO -> /MCU/SWCLK
- U5 pad 11: /Power/INT -> /MCU/INT
- U5 pad 12: /Power/SDA -> /MCU/SDA
- U5 pad 13: /Power/SCL -> /MCU/SCL
- U5 pad 14: /Power/~{CE} -> /MCU/~{CE}
- U5 pad 18: /MCU/VBUS -> /Connectors/VBUS
- U5 pad 3: Net-(RN1-R4.1) -> Net-(U5-*PG)
- U5 pad 6: /Power/TEMP -> /Connectors/TEMP
- U5 pad 8: /Power/V+ -> /Connectors/V+
- U8 pad 53: /MCU/CC2 -> /Connectors/CC2
- U8 pad 54: /MCU/CC2 -> /Connectors/CC2
- U8 pad 70: /MCU/D- -> /Connectors/D-
- U8 pad 71: /MCU/D+ -> /Connectors/D+
- U8 pad 77: /MCU/CC1 -> /Connectors/CC1
- U8 pad 91: /MCU/CC1 -> /Connectors/CC1
Routing:
- net Net-(D1-A): track 0.00 -> 74.6 mm
- net /MCU/KEYPAD.C3: track 0.00 -> 61.2 mm, vias 0 -> 1
- net /MCU/KEYPAD.C2: track 0.00 -> 55.8 mm, vias 0 -> 1
- net /MCU/SCL: track 0.00 -> 44.7 mm, vias 0 -> 3
- net /MCU/KEYPAD.R3: track 0.00 -> 44.5 mm
- net /MCU/~{CE}: track 0.00 -> 42.8 mm, vias 0 -> 3
- net /MCU/INT: track 0.00 -> 42.6 mm, vias 0 -> 3
- net /MCU/SDA: track 0.00 -> 41.3 mm, vias 0 -> 3
- net /Connectors/CC1: track 0.00 -> 37.0 mm, vias 0 -> 3
- net /MCU/SD_IO0: track 0.00 -> 27.8 mm, vias 0 -> 2
- net /Connectors/SDIO.SD_IO0: track 25.2 -> 0.00 mm, vias 2 -> 0
- net /Connectors/SDIO.SD_IO1: track 25.1 -> 0.00 mm, vias 2 -> 0
- net /MCU/SD_IO1: track 0.00 -> 24.8 mm, vias 0 -> 2
- net +3.3V: track 23.7 -> 46.9 mm, vias 5 -> 6
- net /MCU/SD_IO3: track 0.00 -> 15.4 mm
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- added copper zone on F.Cu, net /Connectors/V+
- added copper zone on F.Cu, net /Connectors/VBUS
- added copper zone on B.Cu, net /MCU/KEYPAD.C0
- added copper zone on B.Cu, net /MCU/KEYPAD.C1
- added copper zone on B.Cu, net /MCU/KEYPAD.C2
- added copper zone on B.Cu, net /MCU/KEYPAD.C3
- removed copper zone on F.Cu, net /MCU/VBUS
- removed copper zone on F.Cu, net /Power/V+

Commit message: Getting there part ii
Started power planes, most of keyboard wired together
Parts:
- removed NT1: NetTie_2, NetTie:NetTie-2_SMD_Pad0.5mm
- C17, C35: moved to B.Cu
- SW9: footprint snap dome:snap dome_1 -> snap dome:snap dome_2
- moved R2 175.3 mm to (108.0, 140.1)
- moved C48 33.9 mm to (79.8, 92.0)
- moved C49 33.9 mm to (79.8, 94.8)
- moved C50 33.9 mm to (79.8, 97.5)
- moved C51 33.9 mm to (79.8, 100.2)
- moved C52 33.9 mm to (83.8, 90.9)
- moved C21 22.3 mm to (109.3, 71.1), turned to 180 degrees
- moved C17 16.9 mm to (109.4, 73.2), turned to 180 degrees
- moved C18 16.7 mm to (109.3, 75.3), turned to 180 degrees
- moved U6 9.72 mm to (109.4, 73.2), turned to -90 degrees
- moved R6 8.90 mm to (95.5, 37.0), turned to 90 degrees
- moved C35 2.78 mm to (103.7, 72.0), turned to -90 degrees
- moved C5 2.09 mm to (102.4, 37.0), turned to 90 degrees
- turned SW9 to 0 degrees
Connections:
- net /Misc/MAG1_OUT renamed /MCU/MAG1_OUT
- U8 pad 89: /MCU/SDA -> unconnected-(U8-PB3-Pad89)
- U8 pad 93: /MCU/INT -> /MCU/SDA
- U8 pad 96: unconnected-(U8-PB9-Pad96) -> /MCU/INT
Routing:
- net /MCU/KEYPAD.R0: track 0.00 -> 91.4 mm, vias 0 -> 2
- net Net-(D9-A): track 0.00 -> 90.2 mm
- net Net-(D17-A): track 0.00 -> 85.3 mm, vias 2 -> 3
- net /MCU/KEYPAD.R1: track 0.00 -> 82.3 mm
- net Net-(D13-A): track 0.00 -> 82.0 mm
- net Net-(D8-A): track 0.00 -> 79.2 mm
- net Net-(D7-A): track 0.00 -> 65.5 mm
- net Net-(D16-A): track 0.00 -> 63.4 mm
- net Net-(D15-A): track 0.00 -> 56.3 mm, vias 1 -> 3
- net Net-(D12-A): track 0.00 -> 56.1 mm
- net Net-(D14-A): track 0.00 -> 51.8 mm
- net Net-(D10-A): track 0.00 -> 50.7 mm, vias 1 -> 3
- net Net-(D11-A): track 0.00 -> 47.9 mm
- net /MCU/KEYPAD.R2: track 14.4 -> 54.2 mm, vias 0 -> 4
- net Net-(D6-A): track 0.00 -> 36.2 mm, vias 1 -> 3
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- added copper zone on In1.Cu, net +3.3V
- added copper zone on F.Cu, net /MCU/VDD11C
Other:
- outline, holes or cut-outs redrawn

Commit message: T-2 or 3ish
Just keypad, decaps, and a checkover left!
Parts:
- moved C48 17.8 mm to (63.6, 99.3)
- moved C49 17.8 mm to (63.6, 102.1)
- moved C50 17.8 mm to (63.6, 104.8)
- moved C51 17.8 mm to (63.6, 107.5)
- moved C52 17.8 mm to (67.6, 98.2)
- moved C3 1.54 mm to (112.4, 64.0)
- moved C18 1.21 mm to (109.5, 74.1)
- moved C4 1.21 mm to (112.4, 68.3)
- moved J4 1.21 mm to (109.5, 64.5)
- moved U6 1.21 mm to (109.6, 72.0)
- moved C17 1.21 mm to (109.6, 72.0)
- moved C21 1.21 mm to (109.5, 69.9)
Connections:
- U8 pad 1: unconnected-(U8-PE2-Pad1) -> /Connectors/VCOM
- U8 pad 15: unconnected-(U8-PC0-Pad15) -> /Connectors/R1
- U8 pad 16: unconnected-(U8-PC1-Pad16) -> /Connectors/G1
- U8 pad 17: unconnected-(U8-PC2-Pad17) -> /Connectors/B1
- U8 pad 2: unconnected-(U8-PE3-Pad2) -> /Connectors/GEN
- U8 pad 3: unconnected-(U8-PE4-Pad3) -> /Connectors/GSP
- U8 pad 4: unconnected-(U8-PE5-Pad4) -> /Connectors/GCK
- U8 pad 5: unconnected-(U8-PE6-Pad5) -> /Connectors/INTB
- U8 pad 7: unconnected-(U8-PC13-Pad7) -> /Connectors/BCK
- U8 pad 88: unconnected-(U8-PD7-Pad88) -> /Connectors/B0
- U8 pad 89: unconnected-(U8-PB3-Pad89) -> /Connectors/G0
- U8 pad 90: unconnected-(U8-PB4-Pad90) -> /Connectors/R0
- U8 pad 97: unconnected-(U8-PE0-Pad97) -> /Connectors/BSP
Routing:
- net /Connectors/VCOM: track 0.00 -> 79.6 mm, vias 0 -> 2
- net /Connectors/B0: track 0.00 -> 69.3 mm
- net /Connectors/G0: track 0.00 -> 68.0 mm
- net /Connectors/R0: track 0.00 -> 66.7 mm
- net /Connectors/B1: track 0.00 -> 65.4 mm
- net /Connectors/G1: track 0.00 -> 64.4 mm
- net /Connectors/BSP: track 0.00 -> 63.5 mm
- net /Connectors/R1: track 0.00 -> 63.4 mm
- net /Connectors/GEN: track 0.00 -> 62.3 mm
- net /Connectors/GSP: track 0.00 -> 61.8 mm
- net /Connectors/BCK: track 0.00 -> 56.1 mm
- net /Connectors/INTB: track 0.00 -> 54.7 mm
- net /Connectors/GCK: track 0.00 -> 53.3 mm
- net /Connectors/VA: track 0.00 -> 10.6 mm, vias 0 -> 2
- net unconnected-(U8-PD7-Pad88): track 5.37 -> 0.00 mm, vias 1 -> 0
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
Commit message: Ready to Review
Parts:
- C48, C49, C50, C51, C52: moved to B.Cu
- SW2: footprint Button_Switch_SMD:SW_DIP_SPSTx02_Slide_9.78x7.26mm_W8.61mm_P2.54mm -> Button_Switch_SMD:SW_DIP_SPSTx02_Slide_6.7x6.64mm_W8.61mm_P2.54mm_LowProfile
- moved C52 35.9 mm to (89.1, 127.0), turned to -90 degrees
- moved C51 33.4 mm to (90.7, 127.0), turned to -90 degrees
- moved C50 28.5 mm to (91.7, 109.9)
- moved C48 28.4 mm to (84.6, 118.4)
- moved SW2 26.6 mm to (115.0, 106.5), turned to 90 degrees
- moved C49 25.6 mm to (84.6, 116.7)
- moved D11 18.7 mm to (95.8, 37.8)
- moved D2 15.9 mm to (113.8, 42.9)
- moved D6 10.4 mm to (116.8, 42.9)
- moved D10 9.00 mm to (107.8, 42.9)
- moved D1 7.90 mm to (101.8, 42.9)
- moved D13 7.90 mm to (113.8, 37.8)
- moved D14 7.90 mm to (98.8, 37.8)
- moved D7 7.90 mm to (104.8, 42.9)
- moved D4 6.00 mm to (107.8, 37.8)
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Connections:
- net Net-(J1-SWO) renamed /MCU/SWO
- U8 pad 18: unconnected-(U8-PC3-Pad18) -> /MCU/MAG1_OUT
- U8 pad 22: unconnected-(U8-PA0-Pad22) -> /MCU/KEYPAD.C3
- U8 pad 23: unconnected-(U8-PA1-Pad23) -> /MCU/KEYPAD.C2
- U8 pad 43: unconnected-(U8-PE15-Pad43) -> /MCU/KEYPAD.R0
- U8 pad 44: unconnected-(U8-PB10-Pad44) -> /MCU/KEYPAD.R3
- U8 pad 45: unconnected-(U8-PB11-Pad45) -> /MCU/KEYPAD.R2
- U8 pad 52: unconnected-(U8-PB13-Pad52) -> /MCU/KEYPAD.R1
- U8 pad 81: unconnected-(U8-PD0-Pad81) -> /MCU/KEYPAD.C0
- U8 pad 82: unconnected-(U8-PD1-Pad82) -> /MCU/KEYPAD.C1
Routing:
- net /MCU/KEYPAD.C1: track 0.00 -> 110.3 mm, vias 1 -> 7
- net /MCU/KEYPAD.C0: track 0.00 -> 99.6 mm, vias 1 -> 5
- net /MCU/MAG1_OUT: track 0.00 -> 89.9 mm
- net Net-(IC1-VIN): track 0.65 -> 63.1 mm, vias 5 -> 6
- net /MCU/KEYPAD.C3: track 61.2 -> 111.3 mm, vias 1 -> 7
- net Net-(D13-A): track 82.0 -> 131.6 mm
- net Net-(D12-A): track 56.1 -> 105.5 mm
- net Net-(D4-A): track 27.7 -> 72.8 mm
- net Net-(D11-A): track 47.9 -> 91.9 mm
- net Net-(D5-A): track 28.6 -> 70.8 mm, vias 2 -> 3
- net Net-(D2-A): track 28.4 -> 70.6 mm
- net Net-(D14-A): track 51.8 -> 93.5 mm
- net /MCU/KEYPAD.C2: track 55.8 -> 97.1 mm, vias 1 -> 5
- net Net-(D8-A): track 79.2 -> 120.2 mm
- net Net-(U6-ON/OFF): track 0.00 -> 38.7 mm, vias 0 -> 2
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- removed copper zone on B.Cu, net /MCU/KEYPAD.C0
- removed copper zone on B.Cu, net /MCU/KEYPAD.C1
- removed copper zone on B.Cu, net /MCU/KEYPAD.C2
- removed copper zone on B.Cu, net /MCU/KEYPAD.C3

Commit message: Fixed Obvious Dumb
Parts:
- moved C47 2.55 mm to (88.5, 109.7), turned to 90 degrees
- moved C39 0.41 mm to (105.6, 132.9)
- moved C41 0.07 mm to (107.5, 130.0)
Connections:
- D3 pad 1: /Connectors/D+ -> /Connectors/D-
- D3 pad 3: /Connectors/D- -> /Connectors/D+
- RN1 pad 1: /MCU/SCL -> unconnected-(RN1-R1.1-Pad1)
- RN1 pad 2: /MCU/SDA -> /MCU/SCL
- RN1 pad 3: /MCU/INT -> /MCU/SDA
- RN1 pad 4: unconnected-(RN1-R4.1-Pad4) -> /MCU/INT
Routing:
- net +3.3V: track 64.6 -> 242.1 mm, vias 24 -> 19
- net Net-(D17-A): track 96.1 -> 108.1 mm, vias 3 -> 2
- net /MCU/KEYPAD.R1: track 89.6 -> 82.5 mm, vias 1 -> 5
- net Net-(U5-*PG): track 0.00 -> 6.79 mm
- net Net-(D13-A): track 131.6 -> 138.3 mm
- net Net-(D8-A): track 120.2 -> 114.5 mm, vias 1 -> 2
- net unconnected-(U8-PC6-Pad63): track 7.07 -> 2.46 mm
- net unconnected-(U8-PD15-Pad62): track 6.92 -> 2.68 mm
- net /MCU/SWCLK: track 43.3 -> 39.4 mm
- net unconnected-(U8-PC7-Pad64): track 6.34 -> 2.67 mm
- net unconnected-(U8-PD14-Pad61): track 6.22 -> 2.64 mm
- net /MCU/KEYPAD.R3: track 75.3 -> 78.6 mm
- net unconnected-(U8-PD13-Pad60): track 5.48 -> 2.37 mm
- net unconnected-(U8-PD12-Pad59): track 4.75 -> 1.69 mm
- net unconnected-(U8-PD10-Pad57): track 4.65 -> 1.88 mm
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- removed copper zone on In1.Cu, net +3.3V
- removed copper zone on B.Cu, net /Connectors/VBUS_RAW

Commit message: Production!
Forgot to commit the final, lets hope this works. Also start on software using Slint. Prototype in Plasticity on a free trial to test.
Parts:
- removed SW2: SW_SPST, Button_Switch_SMD:SW_DIP_SPSTx02_Slide_6.7x6.64mm_W8.61mm_P2.54mm_LowProfile
- added C6: 0.1uF, Capacitor_SMD_US_Handsoldering_AKL:C_0603_1608Metric, B.Cu at (106.8, 120.2)
- C17, C3, C35, C4: moved to F.Cu
- C21: value 1uF -> 10uF
- moved C19 8.29 mm to (110.3, 118.8), turned to -90 degrees
- moved C3 5.92 mm to (108.5, 59.5), turned to 0 degrees
- moved C16 4.54 mm to (105.6, 118.6), turned to 90 degrees
- moved C35 3.34 mm to (105.7, 74.7), turned to 180 degrees
- moved C17 2.71 mm to (112.2, 72.8), turned to -90 degrees
- moved C4 1.50 mm to (112.3, 69.8)
Connections:
- C16 pad 1: Net-(IC1-VIN) -> Net-(IC1-CE)
- C17 pad 1: Net-(IC1-VIN) -> Net-(IC1-CE)
- C42 pad 1: Net-(IC1-VIN) -> Net-(IC1-CE)
- IC1 pad 1: Net-(IC1-VIN) -> Net-(IC1-CE)
- L4 pad 1: Net-(IC1-VIN) -> Net-(IC1-CE)
- U5 pad 9: Net-(IC1-VIN) -> Net-(IC1-CE)
- U6 pad 2: Net-(IC1-VIN) -> Net-(IC1-CE)
- U6 pad 5: Net-(U6-ON/OFF) -> Net-(IC1-CE)
Routing:
- net Net-(IC1-VIN): track 62.4 -> 0.00 mm, vias 6 -> 0
- net Net-(IC1-CE): track 19.3 -> 67.8 mm, vias 0 -> 7
- net Net-(U6-ON/OFF): track 38.7 -> 0.00 mm, vias 2 -> 0
- net unconnected-(U8-PE7-Pad35): track 0.00 -> 6.33 mm, vias 0 -> 1
- net unconnected-(U8-PA10-Pad69): track 0.00 -> 5.17 mm, vias 0 -> 1
- net unconnected-(U8-PE8-Pad36): track 0.00 -> 4.37 mm, vias 0 -> 1
- net unconnected-(U8-PA9-Pad68): track 0.00 -> 3.57 mm, vias 0 -> 1
- net unconnected-(U8-PE9-Pad37): track 0.00 -> 3.39 mm, vias 0 -> 1
- net +5V: track 15.0 -> 17.6 mm
- net unconnected-(U8-PA5-Pad29): track 2.64 -> 0.00 mm, vias 1 -> 0
- net unconnected-(U8-PA4-Pad28): track 2.12 -> 0.00 mm, vias 1 -> 0
- net unconnected-(U8-PA8-Pad67): track 0.00 -> 1.83 mm, vias 0 -> 1
- net unconnected-(U8-PD8-Pad55): track 4.60 -> 2.82 mm
- net unconnected-(U8-PD11-Pad58): track 1.57 -> 2.82 mm
- net GND: track 1.04 -> 0.00 mm, vias 257 -> 281
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- added copper zone on B.Cu, net Net-(IC1-CE)
- added copper zone on F.Cu, net Net-(IC1-CE)
- removed copper zone on B.Cu, net Net-(IC1-VIN)
- removed copper zone on F.Cu, net Net-(IC1-VIN)
