File: Hardware/mvpUI/power.kicad_sch (KiCad schematic)
At the start: 23 parts, among them IC1 XC9265B331MR-G, SW2 SW_SPST, U5 BQ25622ERYKR

Commit message: Getting there...
Just need logic and power planes for the most part (and verify everything once more)
Parts:
- added R2: 10k, Resistor_SMD_AKL:R_0603_1608Metric_Pad1.05x0.95mm_HandSolder, symbol Device:R
Connections:
- net +3.3V: now also R2.2
- net at U5.3 (*PG): now also R2.1; no longer RN1.4 (R4.1)
- no-connect marks 2 -> 3

Commit message: Getting there part ii
Started power planes, most of keyboard wired together
Changed lines of the file:
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@@
-    (stroke (width 0) (type default))
-  )
-  (wire (pts (xy 262.89 149.86) (xy 266.7 149.86))
     (stroke (width 0) (type default))
   )
@@
   (label "TEMP" (at 64.77 87.63 180) (fields_autoplaced)
     (effects (font (size 1.27 1.27)) (justify right bottom))
-  )
-  (label "PWR_CLR" (at 266.7 149.86 0) (fields_autoplaced)
-    (effects (font (size 1.27 1.27)) (justify left bottom))
   )
   (label "SDA" (at 138.43 80.01 0) (fields_autoplaced)
@@
   (label "~{CE}" (at 142.24 74.93 180) (fields_autoplaced)
     (effects (font (size 1.27 1.27)) (justify right bottom))
-  )
-  (hierarchical_label "PWR_CLEAR" (shape input) (at 262.89 149.86 180) (fields_autoplaced)
-    (effects (font (size 1.27 1.27)) (justify right))
   )
   (hierarchical_label "{VBAT}" (shape input) (at 54.61 85.09 180) (fields_autoplaced)
@@
   )
   (symbol (lib_id "Device:NetTie_2") (at 262.89 142.875 0) (unit 1)
-    (in_bom no) (on_board yes) (dnp no) (fields_autoplaced)
+    (in_bom no) (on_board no) (dnp no) (fields_autoplaced)
     (property "Reference" "NT1" (at 262.89 138.43 0)
       (effects (font (size 1.27 1.27)))

Commit message: Ready to Review
Parts:
- SW2: footprint Button_Switch_SMD:SW_DIP_SPSTx02_Slide_9.78x7.26mm_W8.61mm_P2.54mm -> Button_Switch_SMD:SW_DIP_SPSTx02_Slide_6.7x6.64mm_W8.61mm_P2.54mm_LowProfile
Changed lines of the file:
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@@
       (effects (font (size 1.27 1.27)))
     )
-    (property "Footprint" "Button_Switch_SMD:SW_DIP_SPSTx02_Slide_9.78x7.26mm_W8.61mm_P2.54mm" (at 224.79 45.72 0)
+    (property "Footprint" "Button_Switch_SMD:SW_DIP_SPSTx02_Slide_6.7x6.64mm_W8.61mm_P2.54mm_LowProfile" (at 224.79 45.72 0)
       (effects (font (size 1.27 1.27)) hide)
     )

Commit message: Fixed Obvious Dumb
Connections:
- net INT: now also RN1.4 (R4.1); no longer RN1.3 (R3.1)
- net SCL: now also RN1.2 (R2.1); no longer RN1.1 (R1.1)
- net SDA: now also RN1.3 (R3.1); no longer RN1.2 (R2.1)
Changed lines of the file:
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@@
   (no_connect (at 91.44 80.01))
   (no_connect (at 137.16 85.09))
-  (no_connect (at 185.42 86.36))
+  (no_connect (at 177.8 86.36))
   (bus_entry (at 41.91 53.34) (size 2.54 2.54)
     (stroke (width 0) (type default))
@@
     (stroke (width 0) (type default))
   )
-  (wire (pts (xy 144.78 93.98) (xy 180.34 93.98))
+  (wire (pts (xy 144.78 93.98) (xy 182.88 93.98))
     (stroke (width 0) (type default))
   )
@@
     (stroke (width 0) (type default))
   )
-  (wire (pts (xy 142.24 96.52) (xy 182.88 96.52))
+  (wire (pts (xy 142.24 96.52) (xy 185.42 96.52))
     (stroke (width 0) (type default))
   )
@@
     (stroke (width 0) (type default))
   )
-  (wire (pts (xy 147.32 91.44) (xy 177.8 91.44))
+  (wire (pts (xy 147.32 91.44) (xy 180.34 91.44))
     (stroke (width 0) (type default))
   )
@@
     (stroke (width 0) (type default))
   )
-  (wire (pts (xy 180.34 93.98) (xy 180.34 86.36))
+  (wire (pts (xy 182.88 93.98) (xy 182.88 86.36))
     (stroke (width 0) (type default))
   )
@@
     (stroke (width 0) (type default))
   )
-  (wire (pts (xy 177.8 91.44) (xy 177.8 86.36))
+  (wire (pts (xy 180.34 91.44) (xy 180.34 86.36))
     (stroke (width 0) (type default))
   )
@@
     (stroke (width 0) (type default))
   )
-  (wire (pts (xy 182.88 96.52) (xy 182.88 86.36))
-    (stroke (width 0) (type default))
-  )
+  (wire (pts (xy 185.42 96.52) (xy 185.42 86.36))
+    (stroke (width 0) (type default))
+  )

Commit message: Production!
Forgot to commit the final, lets hope this works. Also start on software using Slint. Prototype in Plasticity on a free trial to test.
Parts:
- removed SW2: SW_SPST, Button_Switch_SMD:SW_DIP_SPSTx02_Slide_6.7x6.64mm_W8.61mm_P2.54mm_LowProfile, symbol Switch:SW_DIP_x02
- added C6: 0.1uF, Capacitor_SMD_US_Handsoldering_AKL:C_0603_1608Metric, symbol Device:C
- C21: value 1uF -> 10uF
Connections:
- net GND: now also C6.1
- net at C16.1, C17.1, C42.1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: now also IC1.3 (CE), U6.5 (ON/OFF), C6.2
- no-connect marks 3 -> 5
Other:
- moved on the sheet: C17, C21
